Commit message: First changes by Ziyan and Shiyu

File: spot_description/urdf/spot.urdf.xacro (robot description, xacro)
@@ -12,4 +12,9 @@
             </geometry>
         </collision>
+            <inertial>
+      <origin xyz="-0.008399 0.000272 -0.024603"/>
+      <inertia ixx="0.008896" ixy="0.000005" ixz="-0.000193" iyy="0.004922" iyz="0.000033" izz="0.0073030"/>
+      <mass value="1.904699"/>
+    </inertial>
     </link>
     <link name="base_link"/>
@@ -42,4 +47,9 @@
             </geometry>
         </collision>
+            <inertial>
+      <origin xyz="-0.008399 0.000272 -0.024603"/>
+      <inertia ixx="0.008896" ixy="0.000005" ixz="-0.000193" iyy="0.004922" iyz="0.000033" izz="0.0073030"/>
+      <mass value="1.904699"/>
+    </inertial>
     </link>
     <joint name="front_left_hip_x" type="revolute">
@@ -61,4 +71,9 @@
             </geometry>
         </collision>
+            <inertial>
+      <origin xyz="-0.008399 0.000272 -0.024603"/>
+      <inertia ixx="0.008896" ixy="0.000005" ixz="-0.000193" iyy="0.004922" iyz="0.000033" izz="0.0073030"/>
+      <mass value="1.904699"/>
+    </inertial>
     </link>
     <joint name="front_left_hip_y" type="revolute">
@@ -80,4 +95,9 @@
             </geometry>
         </collision>
+            <inertial>
+      <origin xyz="-0.008399 0.000272 -0.024603"/>
+      <inertia ixx="0.008896" ixy="0.000005" ixz="-0.000193" iyy="0.004922" iyz="0.000033" izz="0.0073030"/>
+      <mass value="1.904699"/>
+    </inertial>
     </link>
     <joint name="front_left_knee" type="revolute">
@@ -99,4 +119,9 @@
             </geometry>
         </collision>
+            <inertial>
+      <origin xyz="-0.008399 0.000272 -0.024603"/>
+      <inertia ixx="0.008896" ixy="0.000005" ixz="-0.000193" iyy="0.004922" iyz="0.000033" izz="0.0073030"/>
+      <mass value="1.904699"/>
+    </inertial>
     </link>
     <joint name="front_right_hip_x" type="revolute">
@@ -118,4 +143,9 @@
             </geometry>
         </collision>
+            <inertial>
+      <origin xyz="-0.008399 0.000272 -0.024603"/>
+      <inertia ixx="0.008896" ixy="0.000005" ixz="-0.000193" iyy="0.004922" iyz="0.000033" izz="0.0073030"/>
+      <mass value="1.904699"/>
+    </inertial>
     </link>
     <joint name="front_right_hip_y" type="revolute">
@@ -137,4 +167,9 @@
             </geometry>
         </collision>
+            <inertial>
+      <origin xyz="-0.008399 0.000272 -0.024603"/>
+      <inertia ixx="0.008896" ixy="0.000005" ixz="-0.000193" iyy="0.004922" iyz="0.000033" izz="0.0073030"/>
+      <mass value="1.904699"/>
+    </inertial>
     </link>
     <joint name="front_right_knee" type="revolute">
@@ -156,4 +191,9 @@
             </geometry>
         </collision>
+            <inertial>
+      <origin xyz="-0.008399 0.000272 -0.024603"/>
+      <inertia ixx="0.008896" ixy="0.000005" ixz="-0.000193" iyy="0.004922" iyz="0.000033" izz="0.0073030"/>
+      <mass value="1.904699"/>
+    </inertial>
     </link>
     <joint name="rear_left_hip_x" type="revolute">
@@ -175,4 +215,9 @@
             </geometry>
         </collision>
+            <inertial>
+      <origin xyz="-0.008399 0.000272 -0.024603"/>
+      <inertia ixx="0.008896" ixy="0.000005" ixz="-0.000193" iyy="0.004922" iyz="0.000033" izz="0.0073030"/>
+      <mass value="1.904699"/>
+    </inertial>
     </link>
     <joint name="rear_left_hip_y" type="revolute">
@@ -194,4 +239,9 @@
             </geometry>
         </collision>
+            <inertial>
+      <origin xyz="-0.008399 0.000272 -0.024603"/>
+      <inertia ixx="0.008896" ixy="0.000005" ixz="-0.000193" iyy="0.004922" iyz="0.000033" izz="0.0073030"/>
+      <mass value="1.904699"/>
+    </inertial>
     </link>
     <joint name="rear_left_knee" type="revolute">
@@ -213,4 +263,9 @@
             </geometry>
         </collision>
+            <inertial>
+      <origin xyz="-0.008399 0.000272 -0.024603"/>
+      <inertia ixx="0.008896" ixy="0.000005" ixz="-0.000193" iyy="0.004922" iyz="0.000033" izz="0.0073030"/>
+      <mass value="1.904699"/>
+    </inertial>
     </link>
     <joint name="rear_right_hip_x" type="revolute">
@@ -232,4 +287,9 @@
             </geometry>
         </collision>
+            <inertial>
+      <origin xyz="-0.008399 0.000272 -0.024603"/>
+      <inertia ixx="0.008896" ixy="0.000005" ixz="-0.000193" iyy="0.004922" iyz="0.000033" izz="0.0073030"/>
+      <mass value="1.904699"/>
+    </inertial>
     </link>
     <joint name="rear_right_hip_y" type="revolute">
@@ -251,4 +311,9 @@
             </geometry>
         </collision>
+            <inertial>
+      <origin xyz="-0.008399 0.000272 -0.024603"/>
+      <inertia ixx="0.008896" ixy="0.000005" ixz="-0.000193" iyy="0.004922" iyz="0.000033" izz="0.0073030"/>
+      <mass value="1.904699"/>
+    </inertial>
     </link>
     <joint name="rear_right_knee" type="revolute">
@@ -351,5 +416,5 @@
   </link>
   <joint name="arm_shoulder_0" type="revolute">
-    <parent link="base_link"/>
+    <parent link="body"/>
     <child link="arm0.link_sh0"/>
     <origin xyz="0.292 0.0 0.188"/>
