Commit message: joystick control + publish tf

File: spot_description/urdf/spot_single.urdf.xacro (robot description, xacro)
@@ -2,4 +2,4 @@
     <robot name="spot" xmlns:xacro="http://www.ros.org/wiki/xacro">
     <xacro:include filename="$(find spot_description)/urdf/spot_macro.urdf.xacro" />
-    <xacro:robot_body prefix="spot/"/>
+    <xacro:robot_body prefix="$(arg prefix)/"/>
 </robot>

File: spot_description/urdf/two_spot.urdf.xacro (robot description, xacro)
@@ -4,3 +4,16 @@
     <xacro:robot_body prefix="spot/"/>
     <xacro:robot_body prefix="spot2/"/>
+    <link name="gpe">
+        <origin xyz="0 0 0"/>
+    </link>
+    <joint name="spot/bodyj" type="fixed">
+        <origin xyz="0 0 0" rpy="0 0 0" />
+        <parent link="gpe" />
+        <child link="spot/body" />
+    </joint>
+    <joint name="spot2/bodyj" type="fixed">
+        <origin xyz="0 1 0" rpy="0 0 0" />
+        <parent link="gpe" />
+        <child link="spot2/body" />
+    </joint>
 </robot>
